File: hardware/rpi-cm4-carrier-template/rpi-cm4-carrier-template.kicad_sch (KiCad schematic)
At the start: 0 parts

Commit message: Added dimensions and updated CM4 component properties to include both receptacle options
Other:
- title: Raspberry Pi Compute Module 4 Shoe Template -> Raspberry Pi Compute Module 4 Carrier Template
Changed lines of the file:
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@@
   (paper "A4")
   (title_block
-    (title "Raspberry Pi Compute Module 4 Shoe Template")
+    (title "Raspberry Pi Compute Module 4 Carrier Template")
     (date "2020-10-31")
     (rev "v01")
